File: pedal_uno/pedal_uno.sch (KiCad schematic (older format))
At the start: 22 parts, among them J1 INPUT, P1 Power, P2 Analog, P3 Digital, P4 Digital, P5 CONN_01X01, P6 CONN_01X01, P7 CONN_01X01, P8 CONN_01X01, U1 TL972

Commit message: power
Parts:
- added C? (x3): 6.8n, Capacitor_THT:C_Axial_L5.1mm_D3.1mm_P10.00mm_Horizontal, symbol Device:C
- added C?: 100n, Capacitor_THT:C_Axial_L5.1mm_D3.1mm_P10.00mm_Horizontal, symbol Device:C
- added C? (x2): 4.7u, Capacitor_THT:CP_Radial_D4.0mm_P2.00mm, symbol Device:CP1
- added J?: INPUT, Connector_Audio:Jack_3.5mm_Neutrik_NMJ6HCD2_Horizontal, symbol Connector:Barrel_Jack_Switch
- added R? (x3): 4.7K, Resistor_THT:R_Axial_DIN0207_L6.3mm_D2.5mm_P10.16mm_Horizontal, symbol Device:R
- added R?: 1M2, Resistor_THT:R_Axial_DIN0207_L6.3mm_D2.5mm_P10.16mm_Horizontal, symbol Device:R
- added R? (x2): 100K, Resistor_THT:R_Axial_DIN0207_L6.3mm_D2.5mm_P10.16mm_Horizontal, symbol Device:R
- added U?: TL972, Package_DIP:DIP-8_W7.62mm_LongPads, symbol tl97x:TL972
- C1: value CP1 -> 4.7u
Connections:
- net +2V5: now also C?.1, R?.1, R?.2
- net +5V: now also R?.2
- net GND: now also C?.1, C?.1, C?.2, C?.2, J?.2, J?.3, R?.1, U?.4 (V-)
- net 10(**/SS) renamed PWM_10
- net PWM_10: now also R?.2
- net 9(**) renamed PWM_9
- net PWM_9: now also R?.2
- new net: C?.2, R?.1, R?.1, R?.2
- new net: C?.2, R?.1, R?.2
- new net: C?.2, R?.1, U?.3 (+)
- new net: C?.1, C?.1, U?.1, U?.2 (-)
- new net: C?.1, U?.8 (V+)
- new net: C?.2, J?.1
- no-connect marks 5 -> 12
